File: cm5_io_board_fan_shutdown.kicad_pcb (KiCad board)
At the start: 2 copper layers, 15.5 x 49.5 mm, 33 parts, among them J1 Conn_Pi_JST_SH, J2 Conn_Fan_JST_SH, J3 Conn_Fan_Header, Q1 AO3401A, Q2 BSS138, Q3 BSS138, U1 LM393

Commit message: [update_to_v0.2] Updated version number in silkscreen to revision 0.2, changed QR code to point to project repo
Parts:
- QR*****: value github.com/Eontronics -> GithubQR
Other:
- board text added: "Rev 0.2"
- board text removed: "Rev 0.1"
